File: elec/layout/default/picopixelwall.kicad_pcb (KiCad board)
At the start: 2 copper layers, 225.7 x 100.8 mm, 0 parts

Commit message: working!!!
Parts:
- added C1: 25V 10uF X5R ±10% 0805 Multilayer Ceramic Capacitors MLCC -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, lib:C0805, F.Cu at (63.9, 117.3)
- added C10: 25V 1uF X5R ±10% 0402 Multilayer Ceramic Capacitors MLCC - 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, lib:C0402, F.Cu at (78.1, 107.9)
- added C11: 16V 100nF X7R ±10% 0402 Multilayer Ceramic Capacitors MLCC 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, lib:C0402, F.Cu at (74.4, 114.7)
- added C12: 16V 100nF X7R ±10% 0402 Multilayer Ceramic Capacitors MLCC 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, lib:C0402, F.Cu at (79.7, 116.1)
- added C13: 16V 100nF X7R ±10% 0402 Multilayer Ceramic Capacitors MLCC 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, lib:C0402, F.Cu at (76.7, 126.9)
- added C14: 25V 1uF X5R ±10% 0402 Multilayer Ceramic Capacitors MLCC - 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, lib:C0402, F.Cu at (77.8, 127.0)
- added C15: 16V 100nF X7R ±10% 0402 Multilayer Ceramic Capacitors MLCC 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, lib:C0402, F.Cu at (89.0, 134.7)
- added C16: 16V 100nF X7R ±10% 0402 Multilayer Ceramic Capacitors MLCC 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, lib:C0402, F.Cu at (82.5, 132.7)
- added C17: 16V 100nF X7R ±10% 0402 Multilayer Ceramic Capacitors MLCC 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, lib:C0402, F.Cu at (79.9, 134.8)
- added C18: 16V 100nF X7R ±10% 0402 Multilayer Ceramic Capacitors MLCC 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, lib:C0402, F.Cu at (73.4, 132.7)
- added C19: 16V 100nF X7R ±10% 0402 Multilayer Ceramic Capacitors MLCC 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, lib:C0402, F.Cu at (69.9, 133.1)
- added C2: 25V 10uF X5R ±10% 0805 Multilayer Ceramic Capacitors MLCC -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, lib:C0805, F.Cu at (64.1, 108.3)
- added C20: 16V 100nF X7R ±10% 0402 Multilayer Ceramic Capacitors MLCC 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, lib:C0402, F.Cu at (65.0, 132.7)
- added C21: 16V 100nF X7R ±10% 0402 Multilayer Ceramic Capacitors MLCC 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, lib:C0402, F.Cu at (60.7, 132.8)
- added C22: 16V 100nF X7R ±10% 0402 Multilayer Ceramic Capacitors MLCC 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, lib:C0402, F.Cu at (56.6, 132.9)
- added C23: 16V 100nF X7R ±10% 0402 Multilayer Ceramic Capacitors MLCC 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, lib:C0402, F.Cu at (52.2, 133.1)
- added C24: 16V 100nF X7R ±10% 0402 Multilayer Ceramic Capacitors MLCC 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, lib:C0402, F.Cu at (48.1, 132.8)
- added C25: 50V 10nF X7R ±10% 0402 Multilayer Ceramic Capacitors MLCC -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, lib:C0402, F.Cu at (83.3, 122.8)
- added C3: 50V 20pF C0G ±5% 0402 Multilayer Ceramic Capacitors MLCC - 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, lib:C0402, F.Cu at (70.3, 128.1)
- added C4: 50V 20pF C0G ±5% 0402 Multilayer Ceramic Capacitors MLCC - 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, lib:C0402, F.Cu at (75.6, 128.9)
- added C5: 16V 100nF X7R ±10% 0402 Multilayer Ceramic Capacitors MLCC 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, lib:C0402, F.Cu at (75.7, 126.9)
- added C6: 16V 100nF X7R ±10% 0402 Multilayer Ceramic Capacitors MLCC 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, lib:C0402, F.Cu at (79.7, 117.1)
- added C7: 16V 100nF X7R ±10% 0402 Multilayer Ceramic Capacitors MLCC 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, lib:C0402, F.Cu at (69.1, 116.1)
- added C8: 16V 100nF X7R ±10% 0402 Multilayer Ceramic Capacitors MLCC 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, lib:C0402, F.Cu at (69.1, 117.1)
- added C9: 16V 100nF X7R ±10% 0402 Multilayer Ceramic Capacitors MLCC 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, lib:C0402, F.Cu at (79.8, 120.9)
- added J1: ?, lib:CONN-SMD_4P-P1.00_SM04B-SRSS-TB-LF-SN, F.Cu at (87.1, 128.2)
- added R1: 62.5mW Thick Film Resistors 50V ±100ppm/℃ ±1% 5.1kΩ 0402 Ch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, lib:R0402, F.Cu at (81.2, 111.5)
- added R2: 62.5mW Thick Film Resistors 50V ±100ppm/℃ ±1% 5.1kΩ 0402 Ch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, lib:R0402, F.Cu at (81.1, 108.2)
- added R3: 62.5mW Thick Film Resistors 50V ±100ppm/℃ ±1% 10kΩ 0402 Chi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, lib:R0402, F.Cu at (69.1, 120.9)
- added R4: 62.5mW Thick Film Resistors 50V ±100ppm/℃ ±1% 10kΩ 0402 Chi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, lib:R0402, F.Cu at (71.1, 115.0)
- added R5: 62.5mW Thick Film Resistors 50V ±100ppm/℃ ±1% 1kΩ 0402 Chip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, lib:R0402, F.Cu at (74.2, 125.8)
- added R6: 62.5mW Thick Film Resistors 50V ±100ppm/℃ ±1% 27Ω 0402 Chip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, lib:R0402, F.Cu at (78.1, 114.0)
- added R7: 62.5mW Thick Film Resistors 50V ±100ppm/℃ ±1% 27Ω 0402 Chip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, lib:R0402, F.Cu at (78.1, 115.0)
- added R8: 62.5mW Thick Film Resistors 50V ±100ppm/℃ ±1% 10kΩ 0402 Chi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, lib:R0402, F.Cu at (82.4, 118.0)
- added R9: 62.5mW Thick Film Resistors 50V ±100ppm/℃ ±1% 10kΩ 0402 Chi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, lib:R0402, F.Cu at (83.8, 117.5)
- added U1: ?, lib:USB-C-SMD_KH-TYPE-C-16P, F.Cu at (85.7, 110.0)
- added U10: ?, lib:LED-SMD_4P-L2.0-W2.0-BR, F.Cu at (73.5, 134.8)
- added U11: ?, lib:LED-SMD_4P-L2.0-W2.0-BR, F.Cu at (69.4, 134.8)
- added U12: ?, lib:LED-SMD_4P-L2.0-W2.0-BR, F.Cu at (65.2, 134.8)
- added U13: ?, lib:LED-SMD_4P-L2.0-W2.0-BR, F.Cu at (61.0, 134.8)
- added U14: ?, lib:LED-SMD_4P-L2.0-W2.0-BR, F.Cu at (56.7, 134.8)
- added U15: ?, lib:LED-SMD_4P-L2.0-W2.0-BR, F.Cu at (52.5, 134.8)
- added U16: ?, lib:LED-SMD_4P-L2.0-W2.0-BR, F.Cu at (48.2, 134.9)
- added U17: ?, lib:SOT-23-5_L3.0-W1.7-P0.95-LS2.8-BR, F.Cu at (82.5, 120.5)
- added U2: ?, lib:CONN-TH_XH-2A, F.Cu at (88.2, 119.8)
- added U3: ?, lib:SOT-223-3_L6.5-W3.4-P2.30-LS7.0-BR, F.Cu at (63.9, 112.8)
- added U4: ?, lib:LQFN-56_L7.0-W7.0-P0.4-EP, F.Cu at (74.4, 119.9)
- added U5: ?, lib:OSC-SMD_4P-L3.2-W2.5-BL, F.Cu at (73.0, 128.1)
- added U6: ?, lib:SOIC-8_L5.3-W5.3-P1.27-LS8.0-BL, F.Cu at (74.4, 111.0)
- added U7: ?, lib:LED-SMD_4P-L2.0-W2.0-BR, F.Cu at (86.9, 134.8)
- added U8: ?, lib:LED-SMD_4P-L2.0-W2.0-BR, F.Cu at (82.6, 134.9)
- added U9: ?, lib:LED-SMD_4P-L2.0-W2.0-BR, F.Cu at (77.8, 134.9)
Routing:
- net vcc-1: track 0.00 -> 147.5 mm, vias 0 -> 18
- net vcc-2: track 0.00 -> 79.5 mm, vias 0 -> 5
- net gnd: track 0.00 -> 49.0 mm, vias 0 -> 27
- net gpio2: track 0.00 -> 31.9 mm, vias 0 -> 2
- net micro.micro-vcc: track 0.00 -> 23.5 mm, vias 0 -> 2
- net micro-sck-1: track 0.00 -> 14.4 mm
- net run: track 0.00 -> 13.4 mm, vias 0 -> 2
- net io0: track 0.00 -> 12.8 mm, vias 0 -> 2
- net sda: track 0.00 -> 11.2 mm, vias 0 -> 1
- net scl: track 0.00 -> 10.9 mm, vias 0 -> 1
- net io3: track 0.00 -> 9.73 mm
- net io1: track 0.00 -> 9.57 mm
- net micro-cs-1: track 0.00 -> 9.55 mm
- net dm: track 0.00 -> 8.28 mm
- net xin: track 0.00 -> 8.08 mm
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Other:
- board outline removed
