File: elec/layout/default/picopixelwall.kicad_pcb (KiCad board)
At the start: 2 copper layers, 52 parts, among them J1 ?, U1 ?, U10 ?, U11 ?, U12 ?, U13 ?, U14 ?, U15 ?, U16 ?, U17 ?, U2 ?, U3 ?, U4 ?, U5 ?, U6 ?, U7 ?, U8 ?, U9 ?

Commit message: meters
Parts:
- added C25: 16V 100nF X7R ±10% 0402 Multilayer Ceramic Capacitors MLCC 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, lib:C0402, F.Cu at (39.1, 124.2)
- added C26: 16V 100nF X7R ±10% 0402 Multilayer Ceramic Capacitors MLCC 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, lib:C0402, F.Cu at (44.0, 124.2)
- added C27: 16V 100nF X7R ±10% 0402 Multilayer Ceramic Capacitors MLCC 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, lib:C0402, F.Cu at (49.0, 124.1)
- added C28: 16V 100nF X7R ±10% 0402 Multilayer Ceramic Capacitors MLCC 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, lib:C0402, F.Cu at (54.0, 124.1)
- added C29: 16V 100nF X7R ±10% 0402 Multilayer Ceramic Capacitors MLCC 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, lib:C0402, F.Cu at (59.0, 124.1)
- added C30: 16V 100nF X7R ±10% 0402 Multilayer Ceramic Capacitors MLCC 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, lib:C0402, F.Cu at (64.0, 124.1)
- added C31: 16V 100nF X7R ±10% 0402 Multilayer Ceramic Capacitors MLCC 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, lib:C0402, F.Cu at (69.1, 124.1)
- added C32: 16V 100nF X7R ±10% 0402 Multilayer Ceramic Capacitors MLCC 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, lib:C0402, F.Cu at (74.0, 124.1)
- added C33: 16V 100nF X7R ±10% 0402 Multilayer Ceramic Capacitors MLCC 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, lib:C0402, F.Cu at (79.1, 124.1)
- added C34: 16V 100nF X7R ±10% 0402 Multilayer Ceramic Capacitors MLCC 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, lib:C0402, F.Cu at (83.9, 124.1)
- added U17: ?, lib:LED-SMD_4P-L2.0-W2.0-BR, F.Cu at (38.9, 122.3)
- added U18: ?, lib:LED-SMD_4P-L2.0-W2.0-BR, F.Cu at (43.9, 122.3)
- added U19: ?, lib:LED-SMD_4P-L2.0-W2.0-BR, F.Cu at (48.9, 122.3)
- added U20: ?, lib:LED-SMD_4P-L2.0-W2.0-BR, F.Cu at (53.9, 122.3)
- added U21: ?, lib:LED-SMD_4P-L2.0-W2.0-BR, F.Cu at (58.9, 122.3)
- added U22: ?, lib:LED-SMD_4P-L2.0-W2.0-BR, F.Cu at (63.9, 122.3)
- added U23: ?, lib:LED-SMD_4P-L2.0-W2.0-BR, F.Cu at (68.8, 122.3)
- added U24: ?, lib:LED-SMD_4P-L2.0-W2.0-BR, F.Cu at (73.8, 122.3)
- added U25: ?, lib:LED-SMD_4P-L2.0-W2.0-BR, F.Cu at (78.8, 122.3)
- added U26: ?, lib:LED-SMD_4P-L2.0-W2.0-BR, F.Cu at (83.8, 122.3)
- moved C15 54.0 mm to (39.1, 114.0), turned to 180 degrees
- moved U7 53.1 mm to (38.9, 112.2), turned to 0 degrees
- moved U8 44.9 mm to (43.9, 112.2), turned to 0 degrees
- moved C16 42.8 mm to (44.0, 114.0), turned to 180 degrees
- moved U16 42.3 mm to (83.9, 112.2), turned to 0 degrees
- moved C24 40.5 mm to (83.9, 113.9), turned to 180 degrees
- moved C17 37.3 mm to (49.0, 113.9), turned to 180 degrees
- moved U9 36.8 mm to (48.9, 112.2), turned to 0 degrees
- moved U15 34.8 mm to (78.9, 112.2), turned to 0 degrees
- moved C23 33.0 mm to (79.1, 113.9)
- moved U10 30.0 mm to (53.9, 112.2), turned to 0 degrees
- moved C10 28.7 mm to (106.7, 110.6)
- moved C13 28.7 mm to (105.3, 129.6)
- moved C35 28.7 mm to (112.0, 125.5)
- moved C4 28.7 mm to (104.2, 131.6)
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- renumbered C25 to C35, U17 to U27
Connections:
- net led1.ic-vcc renamed ledrow1.led1.ic-vcc
- net led2.ic-vcc renamed ledrow1.led2.ic-vcc
- net led3.ic-vcc renamed ledrow1.led3.ic-vcc
- net led4.ic-vcc renamed ledrow1.led4.ic-vcc
- net led5.ic-vcc renamed ledrow1.led5.ic-vcc
- net led6.ic-vcc renamed ledrow1.led6.ic-vcc
- net led7.ic-vcc renamed ledrow1.led7.ic-vcc
- net led8.ic-vcc renamed ledrow1.led8.ic-vcc
- net led9.ic-vcc renamed ledrow1.led9.ic-vcc
- U16 pad 2: led10.ic-vcc -> ledrow1-dout
- U2 pad 2: p2 -> gnd
Routing:
- net gnd: track 49.0 -> 335.9 mm, vias 27 -> 54
- net vcc-1: track 147.5 -> 202.7 mm, vias 18 -> 28
- net gpio2: track 31.9 -> 1.41 mm, vias 2 -> 1
- net vcc-2: track 79.5 -> 109.7 mm, vias 5 -> 7
- net ledrow2.led8.ic-vcc: track 0.00 -> 4.24 mm
- net ledrow2.led5.ic-vcc: track 0.00 -> 4.24 mm
- net ledrow2.led4.ic-vcc: track 0.00 -> 4.24 mm
- net ledrow2.led3.ic-vcc: track 0.00 -> 4.24 mm
- net ledrow2.led2.ic-vcc: track 0.00 -> 4.24 mm
- net ledrow2.led9.ic-vcc: track 0.00 -> 4.24 mm
- net ledrow2.led7.ic-vcc: track 0.00 -> 4.24 mm
- net ledrow2.led6.ic-vcc: track 0.00 -> 4.24 mm
- net ledrow1.led5.ic-vcc: track 0.00 -> 4.24 mm
- net ledrow1.led1.ic-vcc: track 2.97 -> 0.00 mm
- net ledrow1.led4.ic-vcc: track 2.80 -> 4.24 mm
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Other:
- board outline added: 84.8 x 38.4 mm
- board text added: "Average Volume"
- board text added: "Live Volume"
