File: elec/src/ams1117-33/elec/layout/default/ams1117-33.kicad_pcb (KiCad board)
At the start: 2 copper layers, 225.7 x 100.8 mm, 3 parts

Commit message: working!!!
Parts:
- moved C1 76.4 mm to (74.3, 124.4), turned to 0 degrees
- moved U1 70.8 mm to (74.4, 119.9), turned to 180 degrees
- moved C2 65.8 mm to (74.5, 115.4), turned to 180 degrees
Routing:
- net gnd: vias 0 -> 3
Other:
- board outline removed
- board text removed: "{{GITHASH}}"
