File: elec/src/rp2040/elec/layout/default/rp2040.kicad_pcb (KiCad board)
At the start: 2 copper layers, 225.7 x 100.8 mm, 20 parts

Commit message: working!!!
Parts:
- moved C1 157.3 mm to (70.3, 128.1)
- moved C10 157.3 mm to (79.7, 116.1)
- moved C11 157.3 mm to (76.7, 126.9)
- moved C12 157.3 mm to (77.8, 127.0)
- moved C2 157.3 mm to (75.6, 128.9)
- moved C3 157.3 mm to (75.7, 126.9)
- moved C4 157.3 mm to (79.7, 117.1)
- moved C5 157.3 mm to (69.1, 116.1)
- moved C6 157.3 mm to (69.1, 117.1)
- moved C7 157.3 mm to (79.8, 120.9)
- moved C8 157.3 mm to (78.1, 107.9)
- moved C9 157.3 mm to (74.4, 114.7)
- moved R1 157.3 mm to (69.1, 120.9)
- moved R2 157.3 mm to (71.1, 115.0)
- moved R3 157.3 mm to (74.2, 125.8)
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Routing:
- net vcc: track 42.5 -> 54.3 mm
Other:
- board outline removed
- board text removed: "{{GITHASH}}"
