File: elec/src/sk6805-ec20/elec/layout/default/sk6805-ec20.kicad_pcb (KiCad board)
At the start: 2 copper layers, 225.7 x 100.8 mm, 2 parts

Commit message: working!!!
Parts:
- moved U1 96.5 mm to (74.4, 119.9), turned to 90 degrees
- moved C1 93.8 mm to (76.5, 119.8), turned to -90 degrees
Other:
- board outline removed
- board text removed: "{{GITHASH}}"
